File: kicad/usb.kicad_sch (KiCad schematic)
At the start: 6 parts, among them J3 USB_C_Receptacle_USB2.0_14P, U5 TPD2EUSB30

Commit message: finish pcb
Parts:
- J3: footprint (none) -> Connector_USB:USB_C_Receptacle_HRO_TYPE-C-31-M-12
- R12, R13, R14, R15: footprint (none) -> Resistor_SMD:R_0805_2012Metric_Pad1.20x1.40mm_HandSolder
Changed lines of the file:
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@@
 	(wire
 		(pts
-			(xy 116.84 46.99) (xy 73.66 46.99)
+			(xy 116.84 46.99) (xy 68.58 46.99)
 		)
 		(stroke
@@
 	(wire
 		(pts
-			(xy 73.66 48.26) (xy 66.04 48.26)
+			(xy 68.58 48.26) (xy 66.04 48.26)
 		)
 		(stroke
@@
 	(wire
 		(pts
-			(xy 73.66 46.99) (xy 73.66 48.26)
+			(xy 68.58 46.99) (xy 68.58 48.26)
 		)
 		(stroke
@@
 			)
 		)
-		(property "Footprint" ""
+		(property "Footprint" "Resistor_SMD:R_0805_2012Metric_Pad1.20x1.40mm_HandSolder"
 			(at 73.66 59.69 0)
 			(effects
@@
 			)
 		)
-		(property "Footprint" ""
+		(property "Footprint" "Resistor_SMD:R_0805_2012Metric_Pad1.20x1.40mm_HandSolder"
 			(at 116.84 50.8 0)
 			(effects
@@
 			)
 		)
-		(property "Footprint" ""
+		(property "Footprint" "Connector_USB:USB_C_Receptacle_HRO_TYPE-C-31-M-12"
 			(at 54.61 55.88 0)
 			(effects
@@
 			)
 		)
-		(property "Footprint" ""
+		(property "Footprint" "Resistor_SMD:R_0805_2012Metric_Pad1.20x1.40mm_HandSolder"
 			(at 73.66 54.61 0)
 			(effects
@@
 			)
 		)
-		(property "Footprint" ""
+		(property "Footprint" "Resistor_SMD:R_0805_2012Metric_Pad1.20x1.40mm_HandSolder"
 			(at 121.92 50.8 0)
 			(effects
